File: poppy/poppy.sch (EAGLE design)
At the start: 5 parts, among them Q1 10MHz

Commit message: Refreshed to encoding
Parts:
- added C3: 4u7, resistor:C-EUC1206K
- added ISP: ISP1, con-lstb:MA03-2
- Q1: device crystal:86SMX -> crystal:CRYSTALCTS406
- renumbered C5 to C1, C6 to C2
Connections:
- new net MISO: ISP.5, U$1.PB3
- new net MOSI: ISP.1, U$1.PB2
- new net N$4: C3.1, U$1.UCAP
- new net RESET: ISP.3, U$1.RESET
- new net SCK: ISP.4, U$1.PB1
- net GND: now also C3.2, ISP.6
- net VCC: now also ISP.2, U$1.AVCC, U$1.UVCC
Changed lines of the file:
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@@
 <classes>
 <class number="0" name="default" width="0" drill="0">
+<clearance class="0" value="0.355"/>
 </class>
 </classes>
@@
 <part name="EDGE" library="mini-pci-e" deviceset="FULL-MINI-PCI-E" device=""/>
 <part name="U$1" library="at90usb" deviceset="AT90USB162" device=""/>
-<part name="Q1" library="crystal" deviceset="86SMX" device="" value="10MHz"/>
-<part name="C5" library="resistor" deviceset="C-EU" device="C1206K" value="22p"/>
-<part name="C6" library="resistor" deviceset="C-EU" device="C1206K" value="22p"/>
+<part name="Q1" library="crystal" deviceset="CRYSTAL" device="CTS406" value="10MHz"/>
+<part name="C1" library="resistor" deviceset="C-EU" device="C1206K" value="22p"/>
+<part name="C2" library="resistor" deviceset="C-EU" device="C1206K" value="22p"/>
 <part name="GND1" library="supply1" deviceset="GND" device=""/>
 <part name="GND2" library="supply1" deviceset="GND" device=""/>
@@
 <part name="GND6" library="supply1" deviceset="GND" device=""/>
 <part name="GND3" library="supply1" deviceset="GND" device=""/>
+<part name="C3" library="resistor" deviceset="C-EU" device="C1206K" value="4u7"/>
+<part name="GND4" library="supply1" deviceset="GND" device=""/>
+<part name="ISP" library="con-lstb" deviceset="MA03-2" device="" value="ISP1"/>
 </parts>
 <sheets>
@@
 <instance part="U$1" gate="G$1" x="-48.26" y="7.62"/>
 <instance part="Q1" gate="G$1" x="-91.44" y="27.94"/>
-<instance part="C5" gate="G$1" x="-99.06" y="20.32"/>
-<instance part="C6" gate="G$1" x="-83.82" y="20.32"/>
+<instance part="C1" gate="G$1" x="-99.06" y="20.32"/>
+<instance part="C2" gate="G$1" x="-83.82" y="20.32"/>
 <instance part="GND1" gate="1" x="-83.82" y="10.16"/>
 <instance part="GND2" gate="1" x="-99.06" y="10.16"/>
@@
 <instance part="GND6" gate="1" x="88.9" y="-30.48"/>
 <instance part="GND3" gate="1" x="-66.04" y="-30.48"/>
+<instance part="C3" gate="G$1" x="-73.66" y="2.54" smashed="yes" rot="R270">
+<attribute name="NAME" x="-77.216" y="-2.159" size="1.778" layer="95"/>
+<attribute name="VALUE" x="-77.216" y="-4.699" size="1.778" layer="96"/>
+</instance>
+<instance part="GND4" gate="1" x="-86.36" y="-2.54"/>
+<instance part="ISP" gate="1" x="-2.54" y="66.04"/>
 </instances>
 <busses>
 <bus name="D+,D-">
 <segment>
-<wire x1="-71.12" y1="-38.1" x2="104.14" y2="-38.1" width="0.762" layer="92"/>
+<wire x1="-81.28" y1="-38.1" x2="104.14" y2="-38.1" width="0.762" layer="92"/>
 <wire x1="104.14" y1="-38.1" x2="104.14" y2="-5.08" width="0.762" layer="92"/>
-<wire x1="-71.12" y1="-38.1" x2="-71.12" y2="-12.7" width="0.762" layer="92"/>
+<wire x1="-81.28" y1="-38.1" x2="-81.28" y2="-12.7" width="0.762" layer="92"/>
+</segment>
+</bus>
+<bus name="MISO,MOSI,SCK,RESET,VCC,GND">
+<segment>
+<wire x1="-20.32" y1="68.58" x2="-20.32" y2="53.34" width="0.762" layer="92"/>
+<wire x1="-20.32" y1="53.34" x2="-20.32" y2="30.48" width="0.762" layer="92"/>
+<wire x1="-20.32" y1="53.34" x2="15.24" y2="53.34" width="0.762" layer="92"/>
+<wire x1="15.24" y1="53.34" x2="15.24" y2="68.58" width="0.762" layer="92"/>
 </segment>
 </bus>
@@
 <segment>
 <pinref part="Q1" gate="G$1" pin="2"/>
-<pinref part="C6" gate="G$1" pin="1"/>
-<wire x1="-86.36" y1="27.94" x2="-83.82" y2="27.94" width="0.1524" layer="91"/>
+<pinref part="C2" gate="G$1" pin="1"/>
+<wire x1="-88.9" y1="27.94" x2="-83.82" y2="27.94" width="0.1524" layer="91"/>
 <wire x1="-83.82" y1="27.94" x2="-83.82" y2="22.86" width="0.1524" layer="91"/>
 <pinref part="U$1" gate="G$1" pin="XTAL2"/>
@@
 <segment>
 <pinref part="Q1" gate="G$1" pin="1"/>
-<pinref part="C5" gate="G$1" pin="1"/>
-<wire x1="-96.52" y1="27.94" x2="-99.06" y2="27.94" width="0.1524" layer="91"/>
+<pinref part="C1" gate="G$1" pin="1"/>
+<wire x1="-93.98" y1="27.94" x2="-99.06" y2="27.94" width="0.1524" layer="91"/>
 <wire x1="-99.06" y1="27.94" x2="-99.06" y2="22.86" width="0.1524" layer="91"/>
 <pinref part="U$1" gate="G$1" pin="XTAL1"/>
@@
 <net name="GND" class="0">
 <segment>
-<pinref part="C6" gate="G$1" pin="2"/>
+<pinref part="C2" gate="G$1" pin="2"/>
 <pinref part="GND1" gate="1" pin="GND"/>
 <wire x1="-83.82" y1="15.24" x2="-83.82" y2="12.7" width="0.1524" layer="91"/>
 </segment>
 <segment>
-<pinref part="C5" gate="G$1" pin="2"/>
+<pinref part="C1" gate="G$1" pin="2"/>
 <pinref part="GND2" gate="1" pin="GND"/>
 <wire x1="-99.06" y1="15.24" x2="-99.06" y2="12.7" width="0.1524" layer="91"/>
@@
 <junction x="-66.04" y="-25.4"/>
 </segment>
+<segment>
+<pinref part="C3" gate="G$1" pin="2"/>
+<pinref part="GND4" gate="1" pin="GND"/>
+<wire x1="-78.74" y1="2.54" x2="-86.36" y2="2.54" width="0.1524" layer="91"/>
+<wire x1="-86.36" y1="2.54" x2="-86.36" y2="0" width="0.1524" layer="91"/>
+</segment>
+<segment>
+<pinref part="ISP" gate="1" pin="6"/>
+<wire x1="-10.16" y1="68.58" x2="-20.32" y2="68.58" width="0.1524" layer="91"/>
+<label x="-15.24" y="68.58" size="1.778" layer="95"/>
+</segment>
 </net>
 <net name="VCC" class="0">
@@
 <wire x1="-63.5" y1="7.62" x2="-71.12" y2="7.62" width="0.1524" layer="91"/>
 </segment>
+<segment>
+<pinref part="U$1" gate="G$1" pin="UVCC"/>
+<wire x1="-63.5" y1="-17.78" x2="-71.12" y2="-17.78" width="0.1524" layer="91"/>
+<label x="-71.12" y="-20.32" size="1.778" layer="95"/>
+</segment>
+<segment>
+<pinref part="U$1" gate="G$1" pin="AVCC"/>
+<wire x1="-63.5" y1="10.16" x2="-71.12" y2="10.16" width="0.1524" layer="91"/>
+<label x="-71.12" y="10.16" size="1.778" layer="95"/>
+</segment>
+<segment>
+<pinref part="ISP" gate="1" pin="2"/>
+<wire x1="-10.16" y1="63.5" x2="-20.32" y2="63.5" width="0.1524" layer="91"/>
+<label x="-15.24" y="63.5" size="1.778" layer="95"/>
+</segment>
 </net>
 <net name="D+" class="0">
@@
 <segment>
 <pinref part="U$1" gate="G$1" pin="D+"/>
-<wire x1="-63.5" y1="-12.7" x2="-71.12" y2="-12.7" width="0.1524" layer="91"/>
-<label x="-66.04" y="-10.16" size="1.778" layer="95" rot="R180"/>
+<wire x1="-63.5" y1="-12.7" x2="-81.28" y2="-12.7" width="0.1524" layer="91"/>
+<label x="-78.74" y="-12.7" size="1.778" layer="95"/>
 </segment>
 </net>
@@
 <segment>
 <pinref part="U$1" gate="G$1" pin="D-"/>
-<wire x1="-63.5" y1="-15.24" x2="-71.12" y2="-15.24" width="0.1524" layer="91"/>
-<label x="-66.04" y="-15.24" size="1.778" layer="95" rot="R180"/>
-</segment>
-</net>
+<wire x1="-63.5" y1="-15.24" x2="-81.28" y2="-15.24" width="0.1524" layer="91"/>
+<label x="-78.74" y="-17.78" size="1.778" layer="95"/>
+</segment>
+</net>
+<net name="N$4" class="0">
+<segment>
+<pinref part="C3" gate="G$1" pin="1"/>
+<pinref part="U$1" gate="G$1" pin="UCAP"/>
+<wire x1="-71.12" y1="2.54" x2="-63.5" y2="2.54" width="0.1524" layer="91"/>
+</segment>
+</net>
+<net name="RESET" class="0">
+<segment>
+<pinref part="U$1" gate="G$1" pin="RESET"/>
+<wire x1="-63.5" y1="38.1" x2="-66.04" y2="38.1" width="0.1524" layer="91"/>
+<wire x1="-66.04" y1="38.1" x2="-66.04" y2="43.18" width="0.1524" layer="91"/>
+<wire x1="-66.04" y1="43.18" x2="-20.32" y2="43.18" width="0.1524" layer="91"/>
+<label x="-63.5" y="43.18" size="1.778" layer="95"/>
+</segment>
+<segment>
+<pinref part="ISP" gate="1" pin="3"/>
+<wire x1="5.08" y1="66.04" x2="15.24" y2="66.04" width="0.1524" layer="91"/>
+<label x="5.08" y="66.04" size="1.778" layer="95"/>
+</segment>
+</net>
+<net name="MOSI" class="0">
+<segment>
+<pinref part="U$1" gate="G$1" pin="PB2"/>
+<wire x1="-33.02" y1="33.02" x2="-20.32" y2="33.02" width="0.1524" layer="91"/>
+<label x="-27.94" y="33.02" size="1.778" layer="95"/>
+</segment>
+<segment>
+<pinref part="ISP" gate="1" pin="1"/>
+<wire x1="5.08" y1="63.5" x2="15.24" y2="63.5" width="0.1524" layer="91"/>
+<label x="5.08" y="63.5" size="1.778" layer="95"/>
+</segment>
+</net>
+<net name="MISO" class="0">
+<segment>
+<pinref part="U$1" gate="G$1" pin="PB3"/>
+<wire x1="-33.02" y1="30.48" x2="-20.32" y2="30.48" width="0.1524" layer="91"/>
+<label x="-27.94" y="30.48" size="1.778" layer="95"/>
+</segment>
+<segment>
+<pinref part="ISP" gate="1" pin="5"/>
+<wire x1="5.08" y1="68.58" x2="15.24" y2="68.58" width="0.1524" layer="91"/>
+<label x="5.08" y="68.58" size="1.778" layer="95"/>
+</segment>
+</net>
+<net name="SCK" class="0">
+<segment>
+<pinref part="U$1" gate="G$1" pin="PB1"/>
+<wire x1="-33.02" y1="35.56" x2="-20.32" y2="35.56" width="0.1524" layer="91"/>
+<label x="-27.94" y="35.56" size="1.778" layer="95"/>
+</segment>
+<segment>
+<pinref part="ISP" gate="1" pin="4"/>
+<wire x1="-10.16" y1="66.04" x2="-20.32" y2="66.04" width="0.1524" layer="91"/>
+<label x="-15.24" y="66.04" size="1.778" layer="95"/>
+</segment>
+</net>

Commit message: Routed
Parts:
- removed U$1: AT90USB162, at90usb:AT90USB162
- added C4: 22p, resistor:C-EUC1206K
- added C5: 4u7, resistor:C-EUC1206K
- added C6: 100n, resistor:C-EUC1206K
- added LED1: LED, led:LEDCHIPLED_0805
- added LED2: CON-RGB-LED-EXT, _led-rgb:CON-RGB-LED-EXT
- added R1: 10k, resistor:R-EU_R1206
- added R2: 1k, resistor:R-EU_R1206
- added R3: 3k9, resistor:R-EU_R1206
- added U1: ATUSB, at90usb:AT90USB162
- added U2: MBI5039, _LedDrivers:MBI5039SOP24-300-1.00
- C1: value 22p -> 100n; device resistor:C-EUC1206K -> resistor:C-EUC4532
- C2: value 22p -> 47u; device resistor:C-EUC1206K -> resistor:CPOL-EU150CLZ-0810
- C3: value 4u7 -> 22p
Connections:
- removed net MOSI: ISP.1, U$1.PB2
- new net LATCH: U1.PB0, U2.LE
- new net MOSI/DATA: ISP.1, U1.PB2, U2.SDI
- new net N$3: LED2.R, U2./OUT0
- new net N$5: LED2.G, U2./OUT1
- new net N$6: LED2.B, U2./OUT2
- new net N$7: LED1.C, R2.2
- new net XTAL1: C3.1, Q1.1, U1.XTAL1
- new net XTAL2: C4.1, Q1.2, U1.XTAL2
- net D+: now also U1.D+; no longer U$1.D+
- net D-: now also U1.D-; no longer U$1.D-
- net GND: now also C2.-, C4.2, C5.2, C6.2, R2.1, R3.1, U1.GND, U1.UGND, U2./OE, U2.GND; no longer C2.2, U$1.GND, U$1.UGND
- net MISO: now also U1.PB3; no longer U$1.PB3
- net N$1: now also LED1.A, U1.PC5; no longer C2.1, Q1.2, U$1.XTAL2
- net N$2: now also R3.2, U2.R-EXT; no longer C1.1, Q1.1, U$1.XTAL1
- net N$4: now also C5.1, U1.UCAP; no longer C3.1, U$1.UCAP
- net RESET: now also R1.1, U1.RESET; no longer U$1.RESET
- net SCK: now also U1.PB1, U2.CLK; no longer U$1.PB1
- net VCC: now also C1.1, C2.+, C6.1, EDGEG$1.3.3V-2, LED2.VCC, R1.2, U1.AVCC, U1.UVCC, U1.VCC, U2.VDD; no longer EDGEG$1.+3.3V-52, U$1.AVCC, U$1.UVCC, U$1.VCC
Other:
- moved on the sheet: C1, C3, ISP, Q1

Commit message: Routed 65%
Connections:
- new net GND18: C3.2, C4.2, EDGEG$1.GND-18
- net GND: no longer C3.2, C4.2
Changed lines of the file:
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@@
 <part name="C3" library="resistor" deviceset="C-EU" device="C1206K" value="22p"/>
 <part name="C4" library="resistor" deviceset="C-EU" device="C1206K" value="22p"/>
-<part name="GND1" library="supply1" deviceset="GND" device=""/>
-<part name="GND2" library="supply1" deviceset="GND" device=""/>
 <part name="GND6" library="supply1" deviceset="GND" device=""/>
 <part name="GND3" library="supply1" deviceset="GND" device=""/>
@@
 <attribute name="VALUE" x="-82.804" y="52.959" size="1.778" layer="96" rot="R180"/>
 </instance>
-<instance part="GND1" gate="1" x="-81.28" y="45.72"/>
-<instance part="GND2" gate="1" x="-96.52" y="45.72"/>
 <instance part="GND6" gate="1" x="-109.22" y="12.7"/>
 <instance part="GND3" gate="1" x="-63.5" y="12.7"/>
@@
 </net>
 <net name="GND" class="0">
-<segment>
-<pinref part="C4" gate="G$1" pin="2"/>
-<pinref part="GND1" gate="1" pin="GND"/>
-<wire x1="-81.28" y1="50.8" x2="-81.28" y2="48.26" width="0.1524" layer="91"/>
-</segment>
-<segment>
-<pinref part="C3" gate="G$1" pin="2"/>
-<pinref part="GND2" gate="1" pin="GND"/>
-<wire x1="-96.52" y1="50.8" x2="-96.52" y2="48.26" width="0.1524" layer="91"/>
-</segment>
 <segment>
 <pinref part="EDGE" gate="G$1" pin="GND-50"/>
@@
 </segment>
 </net>
+<net name="GND18" class="0">
+<segment>
+<pinref part="EDGE" gate="G$1" pin="GND-18"/>
+<wire x1="-121.92" y1="60.96" x2="-114.3" y2="60.96" width="0.1524" layer="91"/>
+<label x="-121.92" y="60.96" size="1.778" layer="95"/>
+</segment>
+<segment>
+<pinref part="C3" gate="G$1" pin="2"/>
+<wire x1="-96.52" y1="50.8" x2="-96.52" y2="45.72" width="0.1524" layer="91"/>
+<label x="-99.06" y="43.18" size="1.778" layer="95"/>
+</segment>
+<segment>
+<pinref part="C4" gate="G$1" pin="2"/>
+<wire x1="-81.28" y1="50.8" x2="-81.28" y2="45.72" width="0.1524" layer="91"/>
+<label x="-83.82" y="43.18" size="1.778" layer="95"/>
+</segment>
+</net>

Commit message: Ready to etch!
Connections:
- removed net GND18: C3.2, C4.2, EDGEG$1.GND-18
- net GND: now also C3.2, C4.2
- net MISO: now also ISP.1; no longer ISP.5
- net MOSI/DATA: now also ISP.4; no longer ISP.1
- net RESET: now also ISP.5; no longer ISP.3
- net SCK: now also ISP.3; no longer ISP.4
Changed lines of the file:
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@@
-</segment>
-<segment>
-<pinref part="ISP" gate="1" pin="6"/>
-<wire x1="33.02" y1="88.9" x2="25.4" y2="88.9" width="0.1524" layer="91"/>
-<label x="27.94" y="88.9" size="1.778" layer="95"/>
 </segment>
 <segment>
@@
 <wire x1="-96.52" y1="88.9" x2="-96.52" y2="91.44" width="0.1524" layer="91"/>
 </segment>
+<segment>
+<pinref part="C3" gate="G$1" pin="2"/>
+<wire x1="-96.52" y1="50.8" x2="-96.52" y2="45.72" width="0.1524" layer="91"/>
+<label x="-99.06" y="43.18" size="1.778" layer="95"/>
+</segment>
+<segment>
+<pinref part="C4" gate="G$1" pin="2"/>
+<wire x1="-81.28" y1="50.8" x2="-81.28" y2="45.72" width="0.1524" layer="91"/>
+<label x="-83.82" y="43.18" size="1.778" layer="95"/>
+</segment>
+<segment>
+<pinref part="ISP" gate="1" pin="6"/>
+<wire x1="33.02" y1="88.9" x2="25.4" y2="88.9" width="0.1524" layer="91"/>
+<label x="25.4" y="88.9" size="1.778" layer="95"/>
+</segment>
 </net>
 <net name="VCC" class="0">
@@
 <pinref part="ISP" gate="1" pin="2"/>
 <wire x1="33.02" y1="83.82" x2="25.4" y2="83.82" width="0.1524" layer="91"/>
-<label x="27.94" y="83.82" size="1.778" layer="95"/>
+<label x="25.4" y="83.82" size="1.778" layer="95"/>
 </segment>
 <segment>
@@
 </segment>
 <segment>
-<pinref part="ISP" gate="1" pin="3"/>
-<wire x1="48.26" y1="86.36" x2="60.96" y2="86.36" width="0.1524" layer="91"/>
-<label x="48.26" y="86.36" size="1.778" layer="95"/>
+<pinref part="ISP" gate="1" pin="5"/>
+<wire x1="48.26" y1="88.9" x2="60.96" y2="88.9" width="0.1524" layer="91"/>
+<label x="48.26" y="88.9" size="1.778" layer="95"/>
 </segment>
 </net>
@@
 </segment>
 <segment>
-<pinref part="ISP" gate="1" pin="5"/>
-<wire x1="48.26" y1="88.9" x2="60.96" y2="88.9" width="0.1524" layer="91"/>
-<label x="48.26" y="88.9" size="1.778" layer="95"/>
+<pinref part="ISP" gate="1" pin="1"/>
+<wire x1="48.26" y1="83.82" x2="60.96" y2="83.82" width="0.1524" layer="91"/>
+<label x="48.26" y="83.82" size="1.778" layer="95"/>
 </segment>
 </net>
@@
 </segment>
 <segment>
-<pinref part="ISP" gate="1" pin="4"/>
-<wire x1="33.02" y1="86.36" x2="25.4" y2="86.36" width="0.1524" layer="91"/>
-<label x="27.94" y="86.36" size="1.778" layer="95"/>
-</segment>
-<segment>
 <pinref part="U2" gate="G$1" pin="CLK"/>
 <wire x1="30.48" y1="50.8" x2="17.78" y2="50.8" width="0.1524" layer="91"/>
 <label x="22.86" y="53.34" size="1.778" layer="95" rot="R180"/>
+</segment>
+<segment>
+<pinref part="ISP" gate="1" pin="3"/>
+<wire x1="48.26" y1="86.36" x2="60.96" y2="86.36" width="0.1524" layer="91"/>
+<label x="48.26" y="86.36" size="1.778" layer="95"/>
 </segment>
 </net>
@@
 </segment>
 <segment>
-<pinref part="ISP" gate="1" pin="1"/>
-<wire x1="48.26" y1="83.82" x2="60.96" y2="83.82" width="0.1524" layer="91"/>
-<label x="48.26" y="83.82" size="1.778" layer="95"/>
-</segment>
-<segment>
 <pinref part="U2" gate="G$1" pin="SDI"/>
 <wire x1="30.48" y1="53.34" x2="17.78" y2="53.34" width="0.1524" layer="91"/>
 <label x="30.48" y="55.88" size="1.778" layer="95" rot="R180"/>
+</segment>
+<segment>
+<pinref part="ISP" gate="1" pin="4"/>
+<wire x1="33.02" y1="86.36" x2="25.4" y2="86.36" width="0.1524" layer="91"/>
+<label x="25.4" y="86.36" size="1.778" layer="95"/>
 </segment>
 </net>
@@
 </segment>
 </net>
-<net name="GND18" class="0">
-<segment>
-<pinref part="EDGE" gate="G$1" pin="GND-18"/>
-<wire x1="-121.92" y1="60.96" x2="-114.3" y2="60.96" width="0.1524" layer="91"/>
-<label x="-121.92" y="60.96" size="1.778" layer="95"/>
-</segment>
-<segment>
-<pinref part="C3" gate="G$1" pin="2"/>
-<wire x1="-96.52" y1="50.8" x2="-96.52" y2="45.72" width="0.1524" layer="91"/>
-<label x="-99.06" y="43.18" size="1.778" layer="95"/>
-</segment>
-<segment>
-<pinref part="C4" gate="G$1" pin="2"/>
-<wire x1="-81.28" y1="50.8" x2="-81.28" y2="45.72" width="0.1524" layer="91"/>
-<label x="-83.82" y="43.18" size="1.778" layer="95"/>
-</segment>
-</net>

Commit message: Layout fixes, testing
Other:
- note added: "Poppy Keyboard Backlight Version 0"
Changed lines of the file:
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@@
 <sheet>
 <plain>
+<frame x1="-208.28" y1="-38.1" x2="106.68" y2="134.62" columns="8" rows="5" layer="94"/>
+<text x="-195.58" y="116.84" size="1.778" layer="94" font="vector">Poppy Keyboard Backlight
+Version 0</text>
 </plain>
 <instances>
@@
 </schematic>
 </drawing>
+<compatibility>
+<note version="6.3" minversion="6.2.2" severity="warning">
+Since Version 6.2.2 text objects can contain more than one line,
+which will not be processed correctly with this version.
+</note>
+</compatibility>
 </eagle>

Commit message: Ready to solder
Parts:
- C1: device resistor:C-EUC4532 -> resistor:C-EUC1206K
- C2: value 47u -> 10u; device resistor:CPOL-EU150CLZ-0810 -> resistor:CPOL-EU153CLV-0807
- C5: value 4u7 -> 1u
- Q1: value 10MHz -> 8MHz; device crystal:CRYSTALCTS406 -> crystal:CSM-7X-DU
- R1, R2: device resistor:R-EU_R1206 -> resistor:R-EU_R3216
- R3: value 3k9 -> 1k; device resistor:R-EU_R1206 -> resistor:R-EU_R3216
Changed lines of the file:
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@@
 <part name="EDGE" library="mini-pci-e" deviceset="FULL-MINI-PCI-E" device="" value=""/>
 <part name="U1" library="at90usb" deviceset="AT90USB162" device="" value="ATUSB"/>
-<part name="Q1" library="crystal" deviceset="CRYSTAL" device="CTS406" value="10MHz"/>
+<part name="Q1" library="crystal" deviceset="CSM-7X-DU" device="" value="8MHz"/>
 <part name="C3" library="resistor" deviceset="C-EU" device="C1206K" value="22p"/>
 <part name="C4" library="resistor" deviceset="C-EU" device="C1206K" value="22p"/>
 <part name="GND6" library="supply1" deviceset="GND" device=""/>
 <part name="GND3" library="supply1" deviceset="GND" device=""/>
-<part name="C5" library="resistor" deviceset="C-EU" device="C1206K" value="4u7"/>
+<part name="C5" library="resistor" deviceset="C-EU" device="C1206K" value="1u"/>
 <part name="GND4" library="supply1" deviceset="GND" device=""/>
 <part name="ISP" library="con-lstb" deviceset="MA03-2" device="" value="ISP1"/>
-<part name="R1" library="resistor" deviceset="R-EU_" device="R1206" value="10k"/>
+<part name="R1" library="resistor" deviceset="R-EU_" device="R3216" value="10k"/>
 <part name="VCC1" library="supply1" deviceset="VCC" device=""/>
 <part name="LED1" library="led" deviceset="LED" device="CHIPLED_0805" value="LED"/>
@@
 <part name="VCC2" library="supply1" deviceset="VCC" device=""/>
 <part name="C6" library="resistor" deviceset="C-EU" device="C1206K" value="100n"/>
-<part name="R3" library="resistor" deviceset="R-EU_" device="R1206" value="3k9"/>
+<part name="R3" library="resistor" deviceset="R-EU_" device="R3216" value="1k"/>
 <part name="GND7" library="supply1" deviceset="GND" device=""/>
 <part name="GND9" library="supply1" deviceset="GND" device=""/>
 <part name="LED2" library="_led-rgb" deviceset="CON-RGB-LED" device="-EXT"/>
 <part name="VCC3" library="supply1" deviceset="VCC" device=""/>
-<part name="R2" library="resistor" deviceset="R-EU_" device="R1206" value="1k"/>
-<part name="C1" library="resistor" deviceset="C-EU" device="C4532" value="100n"/>
+<part name="R2" library="resistor" deviceset="R-EU_" device="R3216" value="1k"/>
+<part name="C1" library="resistor" deviceset="C-EU" device="C1206K" value="100n"/>
 <part name="GND10" library="supply1" deviceset="GND" device=""/>
-<part name="C2" library="resistor" deviceset="CPOL-EU" device="150CLZ-0810" value="47u"/>
+<part name="C2" library="resistor" deviceset="CPOL-EU" device="153CLV-0807" value="10u"/>
 <part name="GND11" library="supply1" deviceset="GND" device=""/>
 </parts>
@@
 </instance>
 <instance part="U1" gate="G$1" x="-45.72" y="50.8"/>
-<instance part="Q1" gate="G$1" x="-88.9" y="60.96" smashed="yes">
+<instance part="Q1" gate="P" x="-88.9" y="60.96" smashed="yes">
 <attribute name="NAME" x="-91.44" y="67.056" size="1.778" layer="95"/>
 <attribute name="VALUE" x="-91.44" y="63.5" size="1.778" layer="96"/>
@@
 <segment>
 <pinref part="C4" gate="G$1" pin="1"/>
-<pinref part="Q1" gate="G$1" pin="2"/>
+<pinref part="Q1" gate="P" pin="2"/>
 <wire x1="-86.36" y1="60.96" x2="-81.28" y2="60.96" width="0.1524" layer="91"/>
 <wire x1="-81.28" y1="60.96" x2="-81.28" y2="58.42" width="0.1524" layer="91"/>
@@
 <pinref part="C3" gate="G$1" pin="1"/>
 <wire x1="-96.52" y1="60.96" x2="-96.52" y2="58.42" width="0.1524" layer="91"/>
-<pinref part="Q1" gate="G$1" pin="1"/>
+<pinref part="Q1" gate="P" pin="1"/>
 <wire x1="-91.44" y1="60.96" x2="-96.52" y2="60.96" width="0.1524" layer="91"/>
 <wire x1="-96.52" y1="60.96" x2="-96.52" y2="71.12" width="0.1524" layer="91"/>
