File: schematic/poppy.sch (EAGLE design)
At the start: 18 parts, among them Q1 8MHz, U1 ATMEGA16U4TQFP44, U2 MBI5030GFSOP-24

Commit message: first production
Parts:
- added LED3: CON-RGB-LED-EXT, _led-rgb:CON-RGB-LED-EXT
- C2: device resistor:CPOL-EU153CLV-0807 -> resistor:C-EUC1812
- Q1: device crystal:CSM-7X-DU -> crystal:CRYSTALCTS406
Connections:
- new net N$11: LED3.R, U2./OUT3
- new net N$12: LED3.G, U2./OUT4
- new net N$13: LED3.B, U2./OUT5
- net GND: now also C2.2; no longer C2.-
- net VCC: now also C2.1, LED3.VCC; no longer C2.+
Changed lines of the file:
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@@
 <parts>
 <part name="EDGE" library="mini-pci-e" deviceset="FULL-MINI-PCI-E" device="" value=""/>
-<part name="Q1" library="crystal" deviceset="CSM-7X-DU" device="" value="8MHz"/>
+<part name="Q1" library="crystal" deviceset="CRYSTAL" device="CTS406" value="8MHz"/>
 <part name="C3" library="resistor" deviceset="C-EU" device="C1206K" value="22p"/>
 <part name="C4" library="resistor" deviceset="C-EU" device="C1206K" value="22p"/>
@@
 <part name="C1" library="resistor" deviceset="C-EU" device="C1206K" value="100n"/>
 <part name="GND10" library="supply1" deviceset="GND" device=""/>
-<part name="C2" library="resistor" deviceset="CPOL-EU" device="153CLV-0807" value="10u"/>
+<part name="C2" library="resistor" deviceset="C-EU" device="C1812" value="10u"/>
 <part name="GND11" library="supply1" deviceset="GND" device=""/>
 <part name="U1" library="p1poppy" deviceset="ATMEGA16U4" device="TQFP44"/>
@@
 <part name="R1" library="resistor" deviceset="R-EU_" device="R1206" value="22"/>
 <part name="R2" library="resistor" deviceset="R-EU_" device="R1206" value="22"/>
+<part name="LED3" library="_led-rgb" deviceset="CON-RGB-LED" device="-EXT"/>
 </parts>
 <sheets>
@@
 <attribute name="VALUE" x="-174.498" y="33.274" size="1.27" layer="94"/>
 </instance>
-<instance part="Q1" gate="P" x="-114.3" y="2.54" smashed="yes">
+<instance part="Q1" gate="G$1" x="-114.3" y="2.54" smashed="yes">
 <attribute name="NAME" x="-116.84" y="8.636" size="1.778" layer="95"/>
 <attribute name="VALUE" x="-116.84" y="5.08" size="1.778" layer="96"/>
@@
 <attribute name="VALUE" x="-90.17" y="37.338" size="1.778" layer="96"/>
 </instance>
+<instance part="LED3" gate="G$1" x="76.2" y="48.26"/>
 </instances>
 <busses>
@@
 <segment>
 <pinref part="C4" gate="G$1" pin="1"/>
-<pinref part="Q1" gate="P" pin="2"/>
+<pinref part="Q1" gate="G$1" pin="2"/>
 <wire x1="-111.76" y1="2.54" x2="-106.68" y2="2.54" width="0.1524" layer="91"/>
 <wire x1="-106.68" y1="2.54" x2="-106.68" y2="0" width="0.1524" layer="91"/>
@@
 <pinref part="C3" gate="G$1" pin="1"/>
 <wire x1="-121.92" y1="2.54" x2="-121.92" y2="0" width="0.1524" layer="91"/>
-<pinref part="Q1" gate="P" pin="1"/>
+<pinref part="Q1" gate="G$1" pin="1"/>
 <wire x1="-116.84" y1="2.54" x2="-121.92" y2="2.54" width="0.1524" layer="91"/>
 <wire x1="-121.92" y1="2.54" x2="-121.92" y2="12.7" width="0.1524" layer="91"/>
@@
 <segment>
 <pinref part="GND11" gate="1" pin="GND"/>
-<pinref part="C2" gate="G$1" pin="-"/>
+<pinref part="C2" gate="G$1" pin="2"/>
 <wire x1="-147.32" y1="-5.08" x2="-147.32" y2="-2.54" width="0.1524" layer="91"/>
 </segment>
@@
 </segment>
 <segment>
-<pinref part="C2" gate="G$1" pin="+"/>
+<pinref part="C2" gate="G$1" pin="1"/>
 <wire x1="-147.32" y1="5.08" x2="-147.32" y2="10.16" width="0.1524" layer="91"/>
 <label x="-147.32" y="12.7" size="1.778" layer="95" rot="R180"/>
@@
 <pinref part="VCC3" gate="VCC" pin="VCC"/>
 <wire x1="93.98" y1="53.34" x2="93.98" y2="63.5" width="0.1524" layer="91"/>
+<pinref part="LED3" gate="G$1" pin="VCC"/>
+<wire x1="93.98" y1="45.72" x2="93.98" y2="53.34" width="0.1524" layer="91"/>
+<junction x="93.98" y="53.34"/>
 </segment>
 </net>
@@
 </segment>
 </net>
+<net name="N$11" class="0">
+<segment>
+<pinref part="U2" gate="MBI5030" pin="/OUT3"/>
+<pinref part="LED3" gate="G$1" pin="R"/>
+<wire x1="66.04" y1="48.26" x2="71.12" y2="48.26" width="0.1524" layer="91"/>
+</segment>
+</net>
+<net name="N$12" class="0">
+<segment>
+<pinref part="U2" gate="MBI5030" pin="/OUT4"/>
+<pinref part="LED3" gate="G$1" pin="G"/>
+<wire x1="66.04" y1="45.72" x2="71.12" y2="45.72" width="0.1524" layer="91"/>
+</segment>
+</net>
+<net name="N$13" class="0">
+<segment>
+<pinref part="U2" gate="MBI5030" pin="/OUT5"/>
+<pinref part="LED3" gate="G$1" pin="B"/>
+<wire x1="66.04" y1="43.18" x2="71.12" y2="43.18" width="0.1524" layer="91"/>
+</segment>
+</net>

Commit message: prod is ready
Connections:
- removed net N$4: C5.1, U1.UCAP
- net VCC: now also C5.1, U1.UCAP; no longer U1.UVCC
Changed lines of the file:
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@@
 <net name="VCC" class="0">
-<segment>
-<wire x1="-55.88" y1="25.4" x2="-68.58" y2="25.4" width="0.1524" layer="91"/>
-<label x="-68.58" y="22.86" size="1.778" layer="95"/>
-<pinref part="U1" gate="U$1" pin="UVCC"/>
-</segment>
 <segment>
 <pinref part="ISP" gate="1" pin="2"/>
@@
 <junction x="93.98" y="53.34"/>
 </segment>
+<segment>
+<pinref part="U1" gate="U$1" pin="UCAP"/>
+<pinref part="C5" gate="G$1" pin="1"/>
+<wire x1="-55.88" y1="45.72" x2="-73.66" y2="45.72" width="0.1524" layer="91"/>
+<wire x1="-73.66" y1="45.72" x2="-73.66" y2="43.18" width="0.1524" layer="91"/>
+<wire x1="-73.66" y1="45.72" x2="-73.66" y2="53.34" width="0.1524" layer="91"/>
+<junction x="-73.66" y="45.72"/>
+<label x="-78.74" y="53.34" size="1.778" layer="95"/>
+<wire x1="-73.66" y1="53.34" x2="-78.74" y2="53.34" width="0.1524" layer="91"/>
+</segment>
 </net>
 <net name="D+" class="0">
@@
 </segment>
 </net>
-<net name="N$4" class="0">
-<segment>
-<pinref part="U1" gate="U$1" pin="UCAP"/>
-<pinref part="C5" gate="G$1" pin="1"/>
-<wire x1="-55.88" y1="45.72" x2="-73.66" y2="45.72" width="0.1524" layer="91"/>
-<wire x1="-73.66" y1="45.72" x2="-73.66" y2="43.18" width="0.1524" layer="91"/>
-</segment>
-</net>
