File: schematic/poppy.brd (EAGLE design)
At the start: 31 x 51.9 mm, 18 parts, among them Q1 8MHz, U1 ATMEGA16U4TQFP44, U2 MBI5030GFSOP-24

Commit message: first production
Parts:
- added LED3: CON-RGB-LED-EXT, _led-rgb:CON-RGB-LED-TH-EXT
- C2: device resistor:153CLV-0807 -> resistor:C1812
- Q1: device crystal:CSM-7X-DU -> crystal:CTS406
- moved R4 24.8 mm to (3.06, 25.2), flipped to the top
- moved LED1 24.7 mm to (2.85, 30.9), flipped to the top
- moved LED2 23.9 mm to (27.0, 36.6), flipped to the top, turned to 180 degrees
- moved R5 21.6 mm to (4.62, 42.2), flipped to the top, turned to 0 degrees
- moved ISP 21.2 mm to (25.4, 10.9), flipped to the top
- moved C6 20.0 mm to (4.92, 36.3), flipped to the top, turned to 180 degrees
- moved C2 19.6 mm to (4.44, 9.35), flipped to the top
- moved Q1 18.2 mm to (17.9, 35.5), flipped to the top, turned to 0 degrees
- moved C1 18.0 mm to (4.04, 18.5), flipped to the top, turned to 180 degrees
- moved C4 14.1 mm to (21.1, 27.5), flipped to the top
- moved C3 13.6 mm to (20.8, 22.0), flipped to the top
- moved C5 11.9 mm to (6.97, 14.9), flipped to the top, turned to 180 degrees
- moved R3 9.92 mm to (17.7, 16.2), flipped to the top, turned to 180 degrees
- moved R2 9.74 mm to (15.0, 9.75), flipped to the top
- moved R1 7.46 mm to (19.0, 9.75), flipped to the top
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Connections:
- new net N$11: LED3.3.R, U2.8
- new net N$12: LED3.2.G, U2.9
- new net N$13: LED3.1.B, U2.10
- net GND: now also C2.2; no longer C2.-
- net VCC: now also C2.1, LED3.4.VCC; no longer C2.+
- net XTAL2: now also Q1.3; no longer Q1.2
Routing:
- net N$11: track 0.00 -> 34.7 mm, vias 0 -> 1
- net GND: track 178.6 -> 146.5 mm, vias 4 -> 0
- net VCC: track 150.9 -> 131.5 mm, vias 0 -> 2
- net N$12: track 0.00 -> 18.3 mm, vias 0 -> 1
- net N$13: track 0.00 -> 17.7 mm
- net SDI: track 5.01 -> 16.3 mm, vias 0 -> 2
- net CLK0: track 15.1 -> 25.0 mm
- net D+: track 15.3 -> 7.95 mm, vias 0 -> 1
- net D-: track 18.3 -> 11.0 mm, vias 0 -> 1
- net DCLK: track 4.92 -> 12.1 mm, vias 0 -> 2
- net RESET: track 24.9 -> 18.1 mm, vias 2 -> 1
- net N$3: track 17.6 -> 22.4 mm, vias 0 -> 1
- net N$4: track 2.53 -> 6.98 mm
- net N$10: track 7.41 -> 11.8 mm, vias 0 -> 2
- net MISO: track 17.6 -> 13.4 mm, vias 0 -> 1
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- added copper zone on layer 1, net GND
- added copper zone on layer 16, net GND
Other:
- board size 31 x 51.9 mm -> 30 x 51 mm

Commit message: prod is ready
Connections:
- removed net N$4: C5.1, U1.6
- net VCC: now also C5.1, U1.6; no longer U1.2
Routing:
- net N$4: track 6.98 -> 0.00 mm
- net VCC: track 131.5 -> 137.9 mm
- net GND: vias 0 -> 4
Changed lines of the file:
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@@
 <vertex x="6" y="44.9"/>
 </polygon>
-<polygon width="0.254" layer="1" isolate="0.6096" orphans="yes">
+<polygon width="0.254" layer="1" isolate="0.6096">
 <vertex x="6" y="50.6"/>
 <vertex x="23.7" y="50.6"/>
@@
 <wire x1="2.9" y1="31.8" x2="3" y2="31.9" width="0.254" layer="1"/>
 <wire x1="3" y1="31.9" x2="4" y2="31.9" width="0.254" layer="1"/>
+<via x="9.5" y="26.2" extent="1-16" drill="0.4"/>
+<via x="13.4" y="45.3" extent="1-16" drill="0.4"/>
+<via x="22.4" y="46.6" extent="1-16" drill="0.4"/>
+<via x="13.8" y="37.9" extent="1-16" drill="0.4"/>
 </signal>
 <signal name="XTAL2">
@@
 <contactref element="C2" pad="1"/>
 <contactref element="EDGE" pad="2"/>
-<contactref element="U1" pad="2"/>
 <contactref element="U1" pad="24"/>
 <contactref element="LED2" pad="4.VCC"/>
@@
 <wire x1="3.5" y1="1.4" x2="3.57" y2="1.32" width="0.254" layer="16"/>
 <wire x1="2.5" y1="9.3" x2="2.49" y2="9.35" width="0.254" layer="1"/>
-<wire x1="8.8" y1="21.7" x2="7.7" y2="21.7" width="0.254" layer="1"/>
+<wire x1="8.9" y1="21.7" x2="7.7" y2="21.7" width="0.254" layer="1"/>
 <wire x1="7.7" y1="21.7" x2="6.7" y2="21.7" width="0.254" layer="1"/>
-<wire x1="8.8" y1="20.4" x2="8.8" y2="21.7" width="0.254" layer="1"/>
 <wire x1="6.7" y1="21.7" x2="6.65" y2="21.75" width="0.254" layer="1"/>
 <wire x1="6.7" y1="19.6" x2="5.6" y2="18.5" width="0.254" layer="1"/>
@@
 <wire x1="20.1" y1="9.8" x2="20.4" y2="10.1" width="0.254" layer="1"/>
 <wire x1="12.7" y1="9.8" x2="20.1" y2="9.8" width="0.254" layer="1"/>
-<wire x1="12.7" y1="19.6" x2="12.7" y2="9.8" width="0.254" layer="1"/>
+<wire x1="12.7" y1="19.6" x2="12.7" y2="18.4" width="0.254" layer="1"/>
+<wire x1="12.7" y1="18.4" x2="12.7" y2="9.8" width="0.254" layer="1"/>
 <wire x1="12.8" y1="19.7" x2="12.7" y2="19.6" width="0.254" layer="1"/>
 <wire x1="12.8" y1="20.4" x2="12.8" y2="19.7" width="0.254" layer="1"/>
@@
 <wire x1="9.9" y1="22.7" x2="8.9" y2="21.7" width="0.254" layer="1"/>
 <wire x1="14.3" y1="22.7" x2="9.9" y2="22.7" width="0.254" layer="1"/>
-<wire x1="8.9" y1="21.7" x2="8.8" y2="21.7" width="0.254" layer="1"/>
 <wire x1="14.3" y1="22.7" x2="14.35" y2="22.65" width="0.254" layer="1"/>
 <wire x1="2.9" y1="9.7" x2="2.6" y2="9.4" width="0.254" layer="1"/>
@@
 <via x="18.9" y="13.1" extent="1-16" drill="0.4"/>
 <wire x1="18.9" y1="13.1" x2="16.3" y2="15.7" width="0.254" layer="1"/>
+<contactref element="U1" pad="6"/>
+<contactref element="C5" pad="1"/>
+<wire x1="12" y1="18.4" x2="12" y2="20.4" width="0.254" layer="1"/>
+<wire x1="8.5" y1="14.9" x2="12" y2="18.4" width="0.254" layer="1"/>
+<wire x1="8.5" y1="14.9" x2="8.47" y2="14.9" width="0.254" layer="1"/>
+<wire x1="12.7" y1="18.4" x2="12" y2="18.4" width="0.254" layer="1"/>
 </signal>
 <signal name="D+">
@@
 <wire x1="9.7" y1="48" x2="9.77" y2="47.92" width="0.254" layer="1"/>
 </signal>
-<signal name="N$4">
-<contactref element="U1" pad="6"/>
-<contactref element="C5" pad="1"/>
-<wire x1="12" y1="18.4" x2="12" y2="20.4" width="0.254" layer="1"/>
-<wire x1="8.5" y1="14.9" x2="12" y2="18.4" width="0.254" layer="1"/>
-<wire x1="8.5" y1="14.9" x2="8.47" y2="14.9" width="0.254" layer="1"/>
-</signal>
 <signal name="N$9">

Commit message: prod is ready 2 lol
Parts:
- moved Q1 1.49 mm to (16.9, 34.4)
Routing:
- net CLK0: track 25.0 -> 18.9 mm
- net SDI: track 16.3 -> 12.7 mm
- net LATCH: track 12.2 -> 9.42 mm
- net XTAL1: track 16.6 -> 14.4 mm
- net N$12: track 18.3 -> 20.4 mm
- net XTAL2: track 18.0 -> 16.7 mm
Changed lines of the file:
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@@
 <elements>
 <element name="EDGE" library="mini-pci-e" package="FULL-MINI-PCI-E" value="" x="11.12" y="-0.13"/>
-<element name="Q1" library="crystal" package="CTS406" value="8MHz" x="17.86" y="35.53" smashed="yes">
-<attribute name="OC_NEWARK" value="unknown" x="34.37" y="-33.05" size="1.778" layer="27" display="off"/>
-<attribute name="MPN" value="" x="34.37" y="-33.05" size="1.778" layer="27" display="off"/>
-<attribute name="MF" value="" x="34.37" y="-33.05" size="1.778" layer="27" display="off"/>
-<attribute name="OC_FARNELL" value="unknown" x="34.37" y="-33.05" size="1.778" layer="27" display="off"/>
-<attribute name="NAME" x="14.43" y="33.92" size="1.27" layer="25" rot="R90"/>
-<attribute name="VALUE" x="15.32" y="31.72" size="1.27" layer="27"/>
+<element name="Q1" library="crystal" package="CTS406" value="8MHz" x="16.86" y="34.43" smashed="yes">
+<attribute name="OC_NEWARK" value="unknown" x="33.37" y="-34.15" size="1.778" layer="27" display="off"/>
+<attribute name="MPN" value="" x="33.37" y="-34.15" size="1.778" layer="27" display="off"/>
+<attribute name="MF" value="" x="33.37" y="-34.15" size="1.778" layer="27" display="off"/>
+<attribute name="OC_FARNELL" value="unknown" x="33.37" y="-34.15" size="1.778" layer="27" display="off"/>
+<attribute name="NAME" x="13.43" y="32.82" size="1.27" layer="25" rot="R90"/>
+<attribute name="VALUE" x="14.32" y="30.62" size="1.27" layer="27"/>
 </element>
 <element name="C3" library="resistor" package="C1206K" value="22p" x="20.835" y="22.025" smashed="yes" rot="R270">
@@
 <wire x1="17.4" y1="25" x2="17.35" y2="24.95" width="0.254" layer="1"/>
 <wire x1="21.1" y1="29" x2="21.06" y2="29.03" width="0.254" layer="1"/>
-<wire x1="21.5" y1="35.3" x2="20.1" y2="36.7" width="0.254" layer="1"/>
-<wire x1="21.5" y1="28.6" x2="21.5" y2="35.3" width="0.254" layer="1"/>
-<wire x1="20.1" y1="36.7" x2="20.06" y2="36.73" width="0.254" layer="1"/>
 <wire x1="21.5" y1="28.6" x2="21.06" y2="29.03" width="0.254" layer="1"/>
 <via x="19.1" y="26.5" extent="1-16" drill="0.4"/>
 <via x="22.5" y="27.5" extent="1-16" drill="0.4"/>
+<wire x1="19.06" y1="35.63" x2="19.17" y2="35.63" width="0.254" layer="1"/>
+<wire x1="19.17" y1="35.63" x2="21" y2="33.8" width="0.254" layer="1"/>
+<wire x1="21" y1="33.8" x2="21" y2="29.09" width="0.254" layer="1"/>
+<wire x1="21" y1="29.09" x2="21.06" y2="29.03" width="0.254" layer="1"/>
 </signal>
 <signal name="XTAL1">
@@
 <wire x1="17.3" y1="25.7" x2="17.35" y2="25.75" width="0.254" layer="1"/>
 <wire x1="20.8" y1="23.6" x2="20.835" y2="23.525" width="0.254" layer="1"/>
-<wire x1="16.8" y1="33.2" x2="15.7" y2="34.3" width="0.254" layer="1"/>
-<wire x1="16.8" y1="32.6" x2="16.8" y2="33.2" width="0.254" layer="1"/>
 <wire x1="16" y1="31.8" x2="16.8" y2="32.6" width="0.254" layer="16"/>
 <wire x1="16" y1="25.7" x2="16" y2="31.8" width="0.254" layer="16"/>
-<wire x1="15.7" y1="34.3" x2="15.66" y2="34.33" width="0.254" layer="1"/>
 <via x="16" y="25.7" extent="1-16" drill="0.4"/>
 <via x="19" y="23.6" extent="1-16" drill="0.4"/>
 <via x="16.8" y="32.6" extent="1-16" drill="0.4"/>
+<wire x1="16" y1="31.8" x2="14.66" y2="33.23" width="0" layer="19" extent="1-16"/>
 </signal>
 <signal name="VCC">
@@
 <contactref element="U1" pad="32"/>
 <contactref element="U2" pad="21"/>
-<wire x1="8.8" y1="30.2" x2="8.8" y2="31.1" width="0.254" layer="1"/>
-<wire x1="9.2" y1="29.8" x2="8.8" y2="30.2" width="0.254" layer="1"/>
-<wire x1="9.2" y1="30.3" x2="9.2" y2="29.8" width="0.254" layer="16"/>
-<wire x1="6.2" y1="33.3" x2="9.2" y2="30.3" width="0.254" layer="16"/>
-<wire x1="6.2" y1="41.8" x2="6.2" y2="33.3" width="0.254" layer="16"/>
-<wire x1="9.4" y1="41.8" x2="6.2" y2="41.8" width="0.254" layer="16"/>
 <wire x1="11.7" y1="44.1" x2="9.4" y2="41.8" width="0.254" layer="1"/>
 <wire x1="11.7" y1="47.9" x2="11.7" y2="44.1" width="0.254" layer="1"/>
 <wire x1="11.7" y1="47.9" x2="11.77" y2="47.92" width="0.254" layer="1"/>
-<via x="9.2" y="29.8" extent="1-16" drill="0.4"/>
 <via x="9.4" y="41.8" extent="1-16" drill="0.4"/>
+<wire x1="9.4" y1="41.8" x2="7.8" y2="40.2" width="0.254" layer="16"/>
+<wire x1="7.8" y1="40.2" x2="7.8" y2="34.3" width="0.254" layer="16"/>
+<via x="7.8" y="34.3" extent="1-16" drill="0.5" diameter="0.254"/>
+<wire x1="7.8" y1="34.3" x2="7.8" y2="33.2" width="0.254" layer="1"/>
+<wire x1="7.8" y1="33.2" x2="8.8" y2="32.2" width="0.254" layer="1"/>
+<wire x1="8.8" y1="32.2" x2="8.8" y2="31.1" width="0.254" layer="1"/>
 </signal>
 <signal name="N$2">
@@
 <wire x1="10.7" y1="29.8" x2="11.2" y2="30.3" width="0.254" layer="1"/>
 <wire x1="10.7" y1="29.7" x2="10.7" y2="29.8" width="0.254" layer="1"/>
-<wire x1="6.9" y1="33.5" x2="10.7" y2="29.7" width="0.254" layer="16"/>
-<wire x1="6.9" y1="38.1" x2="6.9" y2="33.5" width="0.254" layer="16"/>
-<wire x1="9.8" y1="38.1" x2="6.9" y2="38.1" width="0.254" layer="16"/>
 <wire x1="9.8" y1="39.9" x2="9.8" y2="38.1" width="0.254" layer="1"/>
 <wire x1="9.8" y1="39.9" x2="9.77" y2="39.92" width="0.254" layer="1"/>
 <via x="10.7" y="29.7" extent="1-16" drill="0.4"/>
 <via x="9.8" y="38.1" extent="1-16" drill="0.4"/>
+<wire x1="10.7" y1="29.7" x2="9.2" y2="31.2" width="0.254" layer="16"/>
+<wire x1="9.2" y1="31.2" x2="9.2" y2="37.2" width="0.254" layer="16"/>
+<wire x1="9.2" y1="37.2" x2="9.8" y2="37.8" width="0.254" layer="16"/>
+<wire x1="9.8" y1="37.8" x2="9.8" y2="38.1" width="0.254" layer="16"/>
 </signal>
 <signal name="LATCH">
 <contactref element="U1" pad="30"/>
 <contactref element="U2" pad="4"/>
-<wire x1="10.4" y1="32.2" x2="10.4" y2="31.1" width="0.254" layer="1"/>
-<wire x1="7.9" y1="34.7" x2="10.4" y2="32.2" width="0.254" layer="1"/>
-<wire x1="8.2" y1="35" x2="7.9" y2="34.7" width="0.254" layer="16"/>
-<wire x1="9.5" y1="35" x2="8.2" y2="35" width="0.254" layer="16"/>
-<wire x1="11.8" y1="37.3" x2="9.5" y2="35" width="0.254" layer="16"/>
 <wire x1="11.8" y1="39.9" x2="11.8" y2="37.3" width="0.254" layer="1"/>
 <wire x1="11.8" y1="39.9" x2="11.77" y2="39.92" width="0.254" layer="1"/>
-<via x="7.9" y="34.7" extent="1-16" drill="0.4"/>
+<via x="10.4" y="34.4" extent="1-16" drill="0.4"/>
 <via x="11.8" y="37.3" extent="1-16" drill="0.4"/>
+<wire x1="11.8" y1="37.3" x2="10.4" y2="35.9" width="0.254" layer="16"/>
+<wire x1="10.4" y1="35.9" x2="10.4" y2="34.4" width="0.254" layer="16"/>
+<wire x1="10.4" y1="34.4" x2="10.4" y2="31.1" width="0.254" layer="1"/>
 </signal>
 <signal name="N$7">
@@
 <contactref element="U2" pad="9"/>
 <contactref element="LED3" pad="2.G"/>
-<wire x1="16.8" y1="38.1" x2="16.8" y2="39.9" width="0.254" layer="1"/>
-<wire x1="17.4" y1="37.4" x2="16.8" y2="38.1" width="0.254" layer="1"/>
-<wire x1="17.4" y1="35.3" x2="17.4" y2="37.4" width="0.254" layer="1"/>
-<wire x1="26.6" y1="26.1" x2="17.4" y2="35.3" width="0.254" layer="16"/>
-<wire x1="27" y1="26.1" x2="26.6" y2="26.1" width="0.254" layer="16"/>
 <wire x1="16.8" y1="39.9" x2="16.77" y2="39.92" width="0.254" layer="1"/>
-<wire x1="27" y1="26.1" x2="27" y2="26.02" width="0.254" layer="16"/>
-<via x="17.4" y="35.3" extent="1-16" drill="0.4"/>
+<wire x1="27" y1="26.02" x2="26.68" y2="26.02" width="0.254" layer="16"/>
+<wire x1="26.68" y1="26.02" x2="22.4" y2="30.3" width="0.254" layer="16"/>
+<wire x1="22.4" y1="30.3" x2="22.4" y2="35.6" width="0.254" layer="16"/>
+<wire x1="22.4" y1="35.6" x2="20.8" y2="37.2" width="0.254" layer="16"/>
+<wire x1="20.8" y1="37.2" x2="17.4" y2="37.2" width="0.254" layer="16"/>
+<wire x1="17.4" y1="37.2" x2="17" y2="37.6" width="0.254" layer="16"/>
+<via x="17" y="37.6" extent="1-16" drill="0.5" diameter="0.254"/>
+<wire x1="17" y1="37.6" x2="16.77" y2="37.83" width="0.254" layer="1"/>
+<wire x1="16.77" y1="37.83" x2="16.77" y2="39.92" width="0.254" layer="1"/>
 </signal>
 <signal name="N$13">
